File: PCB-files/LidPCB/LidPCB.kicad_pcb (KiCad board)
At the start: 2 copper layers, 1 part, among them J1 Conn_01x25_Female

Commit message: PCB-Push
All parts added
Parts:
- added C1: 100n, Capacitor_SMD:C_0805_2012Metric_Pad1.15x1.40mm_HandSolder, F.Cu at (169.5, 60.8)
- added C2: 100n, Capacitor_SMD:C_0805_2012Metric_Pad1.15x1.40mm_HandSolder, F.Cu at (164.8, 60.8)
- added C3: 4.7u, Resistor_SMD:R_0603_1608Metric_Pad1.05x0.95mm_HandSolder, F.Cu at (158.7, 78.1)
- added C4: 4.7u, Resistor_SMD:R_0603_1608Metric_Pad1.05x0.95mm_HandSolder, F.Cu at (163.2, 74.0)
- added C5: 1u, Capacitor_SMD:C_0805_2012Metric_Pad1.15x1.40mm_HandSolder, F.Cu at (164.8, 63.7)
- added C6: 100n, Capacitor_SMD:C_0805_2012Metric_Pad1.15x1.40mm_HandSolder, F.Cu at (158.9, 65.4)
- added C7: 100n, Capacitor_SMD:C_0805_2012Metric_Pad1.15x1.40mm_HandSolder, F.Cu at (158.9, 68.3)
- added C8: 22pF, Resistor_SMD:R_0603_1608Metric_Pad1.05x0.95mm_HandSolder, F.Cu at (158.7, 75.6)
- added L1: 22uH, LidPCB:IND_LQH2MCN220K02L, F.Cu at (178.3, 60.9)
- added R1: 10k, Resistor_SMD:R_0603_1608Metric_Pad1.05x0.95mm_HandSolder, F.Cu at (167.8, 66.4)
- added R2: 10k, Resistor_SMD:R_0603_1608Metric_Pad1.05x0.95mm_HandSolder, F.Cu at (167.8, 68.9)
- added R3: 10k, Resistor_SMD:R_0603_1608Metric_Pad1.05x0.95mm_HandSolder, F.Cu at (163.4, 68.9)
- added R4: 10k, Resistor_SMD:R_0603_1608Metric_Pad1.05x0.95mm_HandSolder, F.Cu at (169.3, 63.5)
- added R5: 1meg, Resistor_SMD:R_0603_1608Metric_Pad1.05x0.95mm_HandSolder, F.Cu at (163.4, 66.4)
- added R6: 10k, Resistor_SMD:R_0603_1608Metric_Pad1.05x0.95mm_HandSolder, F.Cu at (174.1, 60.5)
- added R7: 140k, Resistor_SMD:R_0603_1608Metric_Pad1.05x0.95mm_HandSolder, F.Cu at (163.2, 71.5)
- added R8: R, Resistor_SMD:R_0603_1608Metric_Pad1.05x0.95mm_HandSolder, F.Cu at (173.7, 63.5)
- added R9: 10k, Resistor_SMD:R_0603_1608Metric_Pad1.05x0.95mm_HandSolder, F.Cu at (194.3, 72.2)
- added U1: XC6206P332MR, Package_TO_SOT_SMD:SOT-23, F.Cu at (158.8, 72.1)
- added U2: R1200N002A-TR-FE, Package_TO_SOT_SMD:SOT-23-6_Handsoldering, F.Cu at (159.4, 61.6)
- added U3: OLED-Display, LidPCB:FPC_Soldering_P0.65x25Pin_OLED, F.Cu at (112.5, 37.5)
- added U4: CAP1293-1-SN, LidPCB:CAP1293-1-SN, F.Cu at (177.6, 82.4)
- J1: value Conn_01x25_Female -> Conn_01x10_Female; footprint Connector_FFC-FPC:FPC_Soldering_P0.65x25Pin_OLED -> muell:686110188622_lid_LIF
- moved J1 59.3 mm to (182.8, 75.5)
Connections:
- J1 pad 1: Net-(J1-Pad1) -> +5V
- J1 pad 2: Net-(J1-Pad2) -> GND
- J1 pad 3: Net-(J1-Pad3) -> SCK
- J1 pad 4: Net-(J1-Pad4) -> DC
- J1 pad 5: Net-(J1-Pad5) -> SDA
- J1 pad 6: Net-(J1-Pad6) -> RST
